Commit message: Adding robot and joint states publishers, rviz visualization

File: resource/storebot.urdf (robot description, URDF)
Before this commit: robot Storebot, 3 links, 2 joints
Links:
- removed link base_footprint
- removed link front_caster
- added link caster wheel; collision box size=0.05 0.028 0.067; visual box size=0.05 0.028 0.067
- added link caster wheel(1); collision box size=0.05 0.028 0.067; visual box size=0.05 0.028 0.067
- added link caster wheel(2); collision box size=0.05 0.028 0.067; visual box size=0.05 0.028 0.067
- added link caster wheel(3); collision box size=0.05 0.028 0.067; visual box size=0.05 0.028 0.067
- added link left_wheel; collision cylinder length=0.095 radius=0.11; visual cylinder length=0.095 radius=0.11
- added link lidar
- added link right_wheel; collision cylinder length=0.095 radius=0.11; visual cylinder length=0.095 radius=0.11
- added link solid; collision cylinder length=0.025 radius=0.0375; visual cylinder length=0.025 radius=0.0375
- added link solid_1; collision cylinder length=0.025 radius=0.0375; visual cylinder length=0.025 radius=0.0375
- added link solid_3; collision cylinder length=0.025 radius=0.0375; visual cylinder length=0.025 radius=0.0375
- added link solid_5; collision cylinder length=0.025 radius=0.0375; visual cylinder length=0.025 radius=0.0375
- link base_link: geometry collision box size=0.1 0.1 0.2; collision box size=0.1 0.1 0.2
Joints:
- removed joint base_joint
- removed joint caster_joint
- added joint CASTER_WHEEL_LF: type continuous, parent base_link, child caster wheel, origin xyz=-0.352 0.45 -0.19 rpy=1.570793 0 2.756718, axis 0 1 0.000003
- added joint CASTER_WHEEL_LR: type continuous, parent base_link, child caster wheel(3), origin xyz=-0.352 -0.45 -0.19 rpy=1.570796 0 -2.821154, axis 0 1 0
- added joint CASTER_WHEEL_RF: type continuous, parent base_link, child caster wheel(1), origin xyz=0.348 0.45 -0.19 rpy=1.570796 0 2.35886, axis 0 1 0
- added joint CASTER_WHEEL_RR: type continuous, parent base_link, child caster wheel(2), origin xyz=0.348 -0.45 -0.19 rpy=1.570796 0 -2.48592, axis 0 1 0
- added joint base_link_lidar_joint: type fixed, parent base_link, child lidar, origin xyz=-0.0001 0 0.12 rpy=0 0 -1.570795
- added joint casterWheelRim: type continuous, parent caster wheel, child solid, origin xyz=0.000003 -0.052101 0.012643 rpy=0.009041 0 0, axis 1 0 0
- added joint casterWheelRim_0: type continuous, parent caster wheel(1), child solid_1, origin xyz=0 -0.052101 0.012643 rpy=-2.695981 0 0, axis 1 0 0
- added joint casterWheelRim_2: type continuous, parent caster wheel(2), child solid_3, origin xyz=-0.000001 -0.052101 0.012643 rpy=0.754265 0 0, axis 1 0 0
- added joint casterWheelRim_4: type continuous, parent caster wheel(3), child solid_5, origin xyz=0 -0.052101 0.012643 rpy=-0.815383 0 0, axis 1 0 0
- added joint left_motor: type continuous, parent base_link, child left_wheel, origin xyz=0.353 0 -0.18 rpy=0.856394 0 0, axis 1 0 0, limit effort=200 velocity=10
- added joint right_motor: type continuous, parent base_link, child right_wheel, origin xyz=-0.3469 0 -0.18 rpy=-1.001909 -0.000002 3.141591, axis -1 -0.000003 0, limit effort=200 velocity=10

Commit message: Adding IMU to URDF model (not shure if needed)

File: resource/storebot.urdf (robot description, URDF)
Before this commit: robot Storebot, 12 links, 11 joints
Links:
- added link imu
Joints:
- added joint base_link_imu_joint: type fixed, parent base_link, child imu, origin xyz=0 0 0 rpy=0 0 0

Commit message: Rotating robot model 90 degree counter clockwise (to make forward along x axis)

File: resource/storebot.urdf (robot description, URDF)
Before this commit: robot /memristor/Documents/storebot.urdf, 13 links, 12 joints
Links:
- link base_link: geometry collision box size=0.1 0.1 0.2; collision box size=0.1 0.1 0.2
Joints:
- joint CASTER_WHEEL_LF: origin xyz=-0.352 0.45 -0.19 rpy=1.570793 0 2.756718 -> xyz=0.45 -0.35 -0.19 rpy=1.570793 0 2.756718
- joint CASTER_WHEEL_LR: origin xyz=-0.352 -0.45 -0.19 rpy=1.570796 0 -2.821154 -> xyz=-0.45 -0.35 -0.19 rpy=1.570796 0 -2.821154
- joint CASTER_WHEEL_RF: origin xyz=0.348 0.45 -0.19 rpy=1.570796 0 2.35886 -> xyz=0.45 0.35 -0.19 rpy=1.570796 0 2.35886
- joint CASTER_WHEEL_RR: origin xyz=0.348 -0.45 -0.19 rpy=1.570796 0 -2.48592 -> xyz=-0.45 0.35 -0.19 rpy=1.570796 0 -2.48592
- joint base_link_lidar_joint: origin xyz=-0.0001 0 0.12 rpy=0 0 -1.570795 -> xyz=0 0 0.12 rpy=0 0 -1.570795
- joint casterWheelRim: origin xyz=0.000003 -0.052101 0.012643 rpy=0.009041 0 0 -> xyz=0 -0.052101 0.012843 rpy=0.009041 0 0
- joint casterWheelRim_0: origin xyz=0 -0.052101 0.012643 rpy=-2.695981 0 0 -> xyz=0 -0.052101 0.012843 rpy=-2.695981 0 0
- joint casterWheelRim_2: origin xyz=-0.000001 -0.052101 0.012643 rpy=0.754265 0 0 -> xyz=0 -0.052101 0.012843 rpy=0.754265 0 0
- joint casterWheelRim_4: origin xyz=0 -0.052101 0.012643 rpy=-0.815383 0 0 -> xyz=0 -0.052101 0.012843 rpy=-0.815383 0 0
- joint left_motor: axis 1 0 0 -> 1 -0.000004 0; origin xyz=0.353 0 -0.18 rpy=0.856394 0 0 -> xyz=0 0.35 -0.18 rpy=0 0 1.5708
- joint right_motor: axis -1 -0.000003 0 -> -1 0.000001 0; origin xyz=-0.3469 0 -0.18 rpy=-1.001909 -0.000002 3.141591 -> xyz=0 -0.35 -0.18 rpy=0 0 -1.570795

Commit message: Lidar and odom finally works in RVIZ. Also deleting caster_wheels from URDF

File: resource/storebot.urdf (robot description, URDF)
Before this commit: robot /memristor/Documents/storebot.urdf, 13 links, 12 joints
Links:
- removed link caster wheel
- removed link caster wheel(1)
- removed link caster wheel(2)
- removed link caster wheel(3)
- removed link solid
- removed link solid_1
- removed link solid_3
- removed link solid_5
- added link base_footprint
- link lidar: geometry collision cylinder length=0.055 radius=0.0508; visual cylinder length=0.055 radius=0.0508
Joints:
- removed joint CASTER_WHEEL_LF
- removed joint CASTER_WHEEL_LR
- removed joint CASTER_WHEEL_RF
- removed joint CASTER_WHEEL_RR
- removed joint base_link_lidar_joint
- removed joint casterWheelRim
- removed joint casterWheelRim_0
- removed joint casterWheelRim_2
- removed joint casterWheelRim_4
- added joint base_joint: type fixed, parent base_link, child base_footprint, origin xyz=0.0 0.0 0.5 rpy=0 0 0
- added joint lidar_joint: type fixed, parent base_link, child lidar, origin xyz=0 0 0.12 rpy=0 0 0
- joint left_motor: type continuous -> fixed
- joint right_motor: type continuous -> fixed

Commit message: Moving footprint down to -0.29

File: resource/storebot.urdf (robot description, URDF)
Before this commit: robot /memristor/Documents/storebot.urdf, 6 links, 5 joints
Joints:
- joint base_joint: origin xyz=0.0 0.0 0.5 rpy=0 0 0 -> xyz=0.0 0.0 -0.29 rpy=0 0 0
